File: MacropadMK.kicad_pcb (KiCad board)
At the start: 4 copper layers, 85.7 x 109.5 mm, 49 parts, among them J4 Qwiic_Vertical, J5 Qwiic_Vertical, SW1 SW_Push, SW10 SW_Push, SW11 SW_Push, SW13 RotaryEncoder_Switch_MP, SW2 SW_Push, SW3 SW_Push, SW4 SW_Push, SW5 SW_Push, SW6 SW_Push, SW7 SW_Push, SW8 SW_Push, SW9 SW_Push

Commit message: first try of layout
Parts:
- added H1: MountingHole, MountingHole:MountingHole_3.2mm_M3, F.Cu at (178.2, 147.3)
- added H2: MountingHole, MountingHole:MountingHole_3.2mm_M3, F.Cu at (104.8, 47.8)
- added H3: MountingHole, MountingHole:MountingHole_3.2mm_M3, F.Cu at (146.2, 86.8)
- added H4: MountingHole, MountingHole:MountingHole_3.2mm_M3, F.Cu at (147.2, 137.3)
- moved C2 128.4 mm to (103.2, 92.3), turned to 90 degrees
- moved D2 85.2 mm to (104.8, 100.3)
- moved R9 82.1 mm to (103.8, 68.6)
- moved D1 78.5 mm to (104.8, 81.3)
- moved D16 78.5 mm to (181.0, 138.4)
- moved D17 78.5 mm to (181.0, 119.4)
- moved R5 61.3 mm to (157.7, 54.8), turned to 0 degrees
- moved R6 61.2 mm to (157.7, 57.3), turned to 0 degrees
- moved R7 61.2 mm to (157.7, 59.8), turned to 0 degrees
- moved R3 58.9 mm to (160.3, 52.3)
- moved R4 58.5 mm to (160.3, 49.8)
- moved C1 50.6 mm to (172.8, 54.3), turned to -90 degrees
- moved C3 50.1 mm to (181.8, 75.8), turned to 0 degrees
- moved D15 38.1 mm to (104.8, 138.4)
- moved D14 38.1 mm to (104.8, 119.4)
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Connections:
- U1 pad 11: unconnected-(U1-GPIO8-Pad11) -> WS12_LED_IN
Routing:
- net ROW3: track 0.00 -> 111.9 mm, vias 0 -> 1
- net ROW2: track 0.00 -> 98.5 mm
- net ROW4: track 0.00 -> 90.4 mm, vias 0 -> 1
- net Net-(D15-DOUT): track 0.00 -> 77.5 mm
- net ROW1: track 0.00 -> 66.7 mm
- net +5V: track 40.0 -> 102.2 mm, vias 0 -> 13
- net COL2: track 57.1 -> 93.1 mm, vias 0 -> 1
- net WS12_LED_IN: track 0.00 -> 34.7 mm
- net COL3: track 57.1 -> 86.4 mm, vias 0 -> 1
- net UART_TX_mmWAVE: track 0.00 -> 28.4 mm, vias 0 -> 1
- net UART_RX_mmWAVE: track 0.00 -> 28.4 mm, vias 0 -> 1
- net Net-(D1-DOUT): track 0.00 -> 25.3 mm
- net Net-(D14-DIN): track 0.00 -> 25.3 mm
- net Net-(D14-DOUT): track 0.00 -> 25.3 mm
- net +3V3: track 10.5 -> 27.3 mm, vias 4 -> 6
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
Commit message: first version with all features
Parts:
- removed R3, R4, R5, R6, R7: 2k2, Resistor_SMD:R_0805_2012Metric
- removed R8: 100R, Resistor_SMD:R_0805_2012Metric
- added F1: Fuse, Fuse:Fuse_0805_2012Metric, B.Cu at (122.2, 149.3)
- added F2: Fuse, Fuse:Fuse_0805_2012Metric, B.Cu at (150.2, 143.8)
- added J1: USB_C_Receptacle_USB2.0_16P_FLAT, Connector_USB:USB_C_Receptacle_HRO_TYPE-C-31-M-12, B.Cu at (130.2, 153.3)
- added J2: USB_C_Receptacle_USB2.0_16P_AXIAL, Connector_USB:USB_C_Receptacle_JAE_DX07S024WJ3R400, B.Cu at (147.5, 148.5)
- added R14: 10k, Resistor_SMD:R_0201_0603Metric, B.Cu at (137.4, 70.8)
- added R15: 10k, Resistor_SMD:R_0201_0603Metric, B.Cu at (173.8, 78.3)
- added R16: 2k2, Resistor_SMD:R_0201_0603Metric, B.Cu at (164.8, 53.8)
- added R17: 2k2, Resistor_SMD:R_0201_0603Metric, B.Cu at (167.8, 53.8)
- added R18: 5k1, Resistor_SMD:R_0201_0603Metric, B.Cu at (121.4, 152.3)
- added R19: 5k1, Resistor_SMD:R_0201_0603Metric, B.Cu at (121.2, 153.8)
- added R20: 5k1, Resistor_SMD:R_0201_0603Metric, B.Cu at (155.8, 150.0)
- added R21: 5k1, Resistor_SMD:R_0201_0603Metric, B.Cu at (147.8, 144.8)
- R10, R12, R13: footprint Resistor_SMD:R_0805_2012Metric -> Resistor_SMD:R_0201_0603Metric
- R11: value 100R -> 10k; footprint Resistor_SMD:R_0805_2012Metric -> Resistor_SMD:R_0201_0603Metric
- R9: footprint Resistor_SMD:R_0805_2012Metric -> Resistor_SMD:R_0603_1608Metric
- moved R11 18.4 mm to (126.8, 66.3)
- moved R13 7.73 mm to (111.1, 59.8)
- moved R12 7.41 mm to (110.8, 52.3)
Connections:
- R11 pad 1: GND -> COL1
- R11 pad 2: Net-(R11-Pad2) -> +3V3
- R12 pad 2: CH_B -> CH_A
- R13 pad 2: CH_A -> CH_B
- SW13 pad C: Net-(R8-Pad1) -> +3V3
- SW13 pad S2: Net-(R11-Pad2) -> GND
Routing:
- net Net-(F2-Pad1): track 0.00 -> 21.3 mm
- net Net-(F1-Pad1): track 0.00 -> 20.9 mm
- net +5V: track 102.2 -> 84.1 mm, vias 13 -> 22
- net Net-(J1-CC1): track 0.00 -> 12.3 mm
- net Net-(J2-CC2): track 0.00 -> 10.7 mm
- net COL3: track 86.4 -> 96.2 mm
- net Net-(J1-CC2): track 0.00 -> 9.15 mm
- net GND: track 0.00 -> 5.85 mm, vias 6 -> 7
- net Net-(R8-Pad1): track 5.20 -> 0.00 mm
- net Net-(R11-Pad2): track 4.67 -> 0.00 mm
- net SDA: track 59.1 -> 56.0 mm
- net COL2: track 93.1 -> 90.8 mm
- net +3V3: track 27.3 -> 25.2 mm, vias 6 -> 9
- net Net-(J2-CC1): track 0.00 -> 1.89 mm
- net CH_A: track 34.7 -> 36.0 mm
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Other:
- board size 85.7 x 109.5 mm -> 85.7 x 114.3 mm

Commit message: ready to order, all features prepared
Parts:
- added H5: MountingHole, MountingHole:MountingHole_3.2mm_M3, F.Cu at (105.8, 152.5)
- added J3: Conn_01x03_Pin, Connector_JST:JST_SH_BM03B-SRSS-TB_1x03-1MP_P1.00mm_Vertical, B.Cu at (105.0, 59.6)
- added J6: Conn_01x03_Pin, Connector_JST:JST_SH_BM03B-SRSS-TB_1x03-1MP_P1.00mm_Vertical, B.Cu at (111.2, 68.1)
- added J7: Conn_01x03_Pin, Connector_JST:JST_SH_BM03B-SRSS-TB_1x03-1MP_P1.00mm_Vertical, B.Cu at (161.6, 53.8)
- added R23: 10k, Resistor_SMD:R_0201_0603Metric, B.Cu at (109.1, 57.3)
- added R24: 10k, Resistor_SMD:R_0201_0603Metric, B.Cu at (110.8, 57.3)
- added R25: 10k, Resistor_SMD:R_0201_0603Metric, B.Cu at (110.2, 63.3)
- added R26: 10k, Resistor_SMD:R_0201_0603Metric, B.Cu at (112.4, 63.3)
- added R27: 10k, Resistor_SMD:R_0201_0603Metric, B.Cu at (157.8, 52.6)
- added R28: 10k, Resistor_SMD:R_0201_0603Metric, B.Cu at (157.8, 55.1)
- moved H4 16.5 mm to (148.2, 120.8)
- moved H1 4.12 mm to (179.2, 151.3)
Connections:
- U1 pad 19: unconnected-(U1-GPIO45-Pad19) -> GPIO45
- U1 pad 20: unconnected-(U1-GPIO42-Pad20) -> GPIO42
- U1 pad 21: unconnected-(U1-GPIO41-Pad21) -> GPIO41
Routing:
- net GPIO42: track 0.00 -> 62.6 mm
- net GPIO41: track 0.00 -> 56.8 mm, vias 0 -> 3
- net GPIO45: track 0.00 -> 13.3 mm, vias 0 -> 1
- net +3V3: track 25.2 -> 35.5 mm, vias 9 -> 13
- net COL3: track 96.2 -> 92.7 mm

Commit message: add light sensor
Parts:
- added C4: 100n, Capacitor_SMD:C_0805_2012Metric, B.Cu at (119.0, 45.4)
- added Q1: BPW85, LED_SMD:LED_0603_1608Metric, B.Cu at (115.0, 45.4)
- added R29: 100k, Resistor_SMD:R_0603_1608Metric, B.Cu at (113.3, 47.7)
- R10, R11, R12, R13, R14, R15, R16, R17, R18, R19, R20, R21, R23, R24, R25, R26, R27, R28: footprint Resistor_SMD:R_0201_0603Metric -> Resistor_SMD:R_0603_1608Metric
- moved R13 3.62 mm to (113.5, 57.1), turned to -90 degrees
- moved H2 2.20 mm to (106.2, 49.5)
- moved H1 1.30 mm to (178.8, 150.1)
- moved R11 1.14 mm to (126.5, 67.4)
- moved R25 1.08 mm to (109.2, 63.3)
- moved R21 1.04 mm to (147.4, 143.8)
- moved R27 1.00 mm to (156.8, 52.6)
- moved R28 0.96 mm to (157.7, 56.1)
- moved R16 0.80 mm to (165.6, 53.8)
- moved R17 0.80 mm to (168.6, 53.8)
- moved R24 0.76 mm to (111.5, 57.0), turned to -90 degrees
- moved R18 0.70 mm to (121.5, 151.6)
- moved R19 0.64 mm to (121.5, 154.4)
- moved H5 0.52 mm to (105.2, 152.4)
- moved R23 0.34 mm to (109.0, 57.0), turned to 90 degrees
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Connections:
- U1 pad 24: unconnected-(U1-GPIO38-Pad24) -> Brightness
Routing:
- net +5V: track 84.1 -> 308.3 mm, vias 22 -> 14
- net +3V3: track 35.5 -> 188.9 mm, vias 13 -> 5
- net Brightness: track 0.00 -> 46.4 mm, vias 0 -> 3
- net GND: track 5.85 -> 23.4 mm, vias 7 -> 12
- net GPIO42: track 62.6 -> 49.1 mm, vias 0 -> 1
- net Net-(F2-Pad1): track 21.3 -> 14.1 mm
- net CH_B: track 26.8 -> 24.0 mm
- net COL1: track 110.1 -> 111.6 mm
- net SDA: track 56.0 -> 54.8 mm
- net COL2: track 90.8 -> 90.2 mm
- net Net-(J2-CC1): track 1.89 -> 2.51 mm
- net COL3: track 92.7 -> 92.2 mm
- removed copper zone on In1.Cu, net +3V3
- removed copper zone on In2.Cu, net +5V
Other:
- copper layers 4 -> 2
- board text added: "MacropadMK_1"
