File: MacropadMK.kicad_sch (KiCad schematic)
At the start: 69 parts, among them J1 USB_C_Receptacle_USB2.0_16P_F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, J2 USB_C_Receptacle_USB2.0_16P_A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, J3 Conn_01x03_Pin, J4 Qwiic_Vertical, J5 Qwiic_Vertical, J6 Conn_01x03_Pin, J7 Conn_01x03_Pin, SW1 SW_Push, SW10 SW_Push, SW11 SW_Push, SW13 RotaryEncoder_Switch_MP, SW2 SW_Push, SW3 SW_Push, SW4 SW_Push, SW5 SW_Push, SW6 SW_Push, SW7 SW_Push, SW8 SW_Push, SW9 SW_Push

Commit message: add light sensor
Parts:
- added C4: 100n, Capacitor_SMD:C_0805_2012Metric, symbol Device:C
- added Q1: BPW85, LED_SMD:LED_0603_1608Metric, symbol Sensor_Optical:BPW85
- added R29: 100k, Resistor_SMD:R_0603_1608Metric, symbol Device:R
- R10, R11, R12, R13, R14, R15, R16, R17, R18, R19, R20, R21, R23, R24, R25, R26, R27, R28: footprint Resistor_SMD:R_0201_0603Metric -> Resistor_SMD:R_0603_1608Metric
Connections:
- net +3V3: now also R29.2
- net GND: now also C4.2, Q1.2 (E)
- net Brightness: now reaches U1.24 (GPIO38)
- net Brightness: now also C4.1, Q1.1 (C), R29.1
